File: hardware/usb-redriver/usb-redriver.kicad_sch (KiCad schematic)
At the start: 33 parts, among them J1 USB3 IN, J2 USB3 OUT, U1 PTN36241BBS, U2 SE8119AKN

Commit message: Assign part numbers and footprints to USB connectors
Parts:
- J1: footprint (none) -> Connector_USB:USB3_A_Plug_Wuerth_692112030100_Horizontal; MFR (none) -> Wurth; MPN (none) -> 692112030100
- J2: footprint (none) -> Connector_USB:USB3_A_Receptacle_Wuerth_692122030100; MFR (none) -> Wurth; MPN (none) -> 692122030100
Changed lines of the file:
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@@
 			)
 		)
-		(property "Footprint" ""
+		(property "Footprint" "Connector_USB:USB3_A_Plug_Wuerth_692112030100_Horizontal"
 			(at 50.8 50.8 0)
 			(effects
@@
 			)
 		)
+		(property "MFR" "Wurth"
+			(at 46.99 53.34 0)
+			(effects
+				(font
+					(size 1.27 1.27)
+				)
+				(hide yes)
+			)
+		)
+		(property "MPN" "692112030100"
+			(at 46.99 53.34 0)
+			(effects
+				(font
+					(size 1.27 1.27)
+				)
+				(hide yes)
+			)
+		)
 		(pin "9"
 		)
@@
 			)
 		)
-		(property "Footprint" ""
+		(property "Footprint" "Connector_USB:USB3_A_Receptacle_Wuerth_692122030100"
 			(at 50.8 109.22 0)
 			(effects
@@
 			(at 46.99 111.76 0)
 			(effects
+				(font
+					(size 1.27 1.27)
+				)
+				(hide yes)
+			)
+		)
+		(property "MFR" "Wurth"
+			(at 46.99 111.76 0)
+			(effects
+				(font
+					(size 1.27 1.27)
+				)
+				(hide yes)
+			)
+		)
+		(property "MPN" "692122030100"
+			(at 46.99 111.76 0)
+			(effects

Commit message: Use local USB connector footprints to pair with 3D models
Parts:
- J1: footprint Connector_USB:USB3_A_Plug_Wuerth_692112030100_Horizontal -> local_connector_usb:USB3_A_Plug_Wuerth_692112030100_Horizontal
- J2: footprint Connector_USB:USB3_A_Receptacle_Wuerth_692122030100 -> local_connector_usb:USB3_A_Receptacle_Wuerth_692122030100
Changed lines of the file:
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@@
 			)
 		)
-		(property "Footprint" "Connector_USB:USB3_A_Plug_Wuerth_692112030100_Horizontal"
+		(property "Footprint" "local_connector_usb:USB3_A_Plug_Wuerth_692112030100_Horizontal"
 			(at 50.8 50.8 0)
 			(effects
@@
 			)
 		)
-		(property "Footprint" "Connector_USB:USB3_A_Receptacle_Wuerth_692122030100"
+		(property "Footprint" "local_connector_usb:USB3_A_Receptacle_Wuerth_692122030100"
 			(at 50.8 109.22 0)
 			(effects

Commit message: Transfer values for capacitors
Parts:
- C1, C2, C9: value C -> 2u2; footprint (none) -> Capacitor_SMD:C_0805_2012Metric
- C10, C12, C13, C15, C3, C4, C5, C6, C7, C8: value C -> 100n; footprint (none) -> Capacitor_SMD:C_0402_1005Metric
- C11, C14: value C -> 22u; footprint (none) -> Capacitor_SMD:C_1206_3216Metric
Other:
- moved on the sheet: C10, C11, C12, C15, C2, C3

Commit message: Transfer values for resistors
Parts:
- R10, R13, R14, R2, R3, R4, R8, R9: now not fitted
- R12: value 44k5 -> 75k
- R6: value 38k -> 75k
Changed lines of the file:
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@@
 			)
 		)
-		(property "Value" "38k"
+		(property "Value" "75k"
 			(at 134.62 88.8999 0)
 			(effects
@@
 		(in_bom yes)
 		(on_board yes)
-		(dnp no)
+		(dnp yes)
 		(fields_autoplaced yes)
 		(property "Reference" "R2"
@@
 		(in_bom yes)
 		(on_board yes)
-		(dnp no)
+		(dnp yes)
 		(fields_autoplaced yes)
 		(property "Reference" "R9"
@@
 		(in_bom yes)
 		(on_board yes)
-		(dnp no)
+		(dnp yes)
 		(fields_autoplaced yes)
 		(property "Reference" "R14"
@@
 		(in_bom yes)
 		(on_board yes)
-		(dnp no)
+		(dnp yes)
 		(fields_autoplaced yes)
 		(property "Reference" "R13"
@@
 			)
 		)
-		(property "Value" "44k5"
+		(property "Value" "75k"
 			(at 165.1 111.7599 0)
 			(effects
@@
 		(in_bom yes)
 		(on_board yes)
-		(dnp no)
+		(dnp yes)
 		(fields_autoplaced yes)
 		(property "Reference" "R8"
@@
 		(in_bom yes)
 		(on_board yes)
-		(dnp no)
+		(dnp yes)
 		(fields_autoplaced yes)
 		(property "Reference" "R3"
@@
 		(in_bom yes)
 		(on_board yes)
-		(dnp no)
+		(dnp yes)
 		(fields_autoplaced yes)
 		(property "Reference" "R10"
@@
 		(in_bom yes)
 		(on_board yes)
-		(dnp no)
+		(dnp yes)
 		(fields_autoplaced yes)
 		(property "Reference" "R4"

Commit message: Assign footprints for resistors
Parts:
- R1, R10, R11, R12, R13, R14, R2, R3, R4, R5, R6, R7, R8, R9: footprint (none) -> Resistor_SMD:R_0402_1005Metric
Changed lines of the file:
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@@
 			)
 		)
-		(property "Footprint" ""
+		(property "Footprint" "Resistor_SMD:R_0402_1005Metric"
 			(at 112.522 69.85 90)
 			(effects
@@
 			)
 		)
-		(property "Footprint" ""
+		(property "Footprint" "Resistor_SMD:R_0402_1005Metric"
 			(at 151.892 110.49 90)
 			(effects
@@
 			)
 		)
-		(property "Footprint" ""
+		(property "Footprint" "Resistor_SMD:R_0402_1005Metric"
 			(at 130.302 87.63 90)
 			(effects
@@
 			)
 		)
-		(property "Footprint" ""
+		(property "Footprint" "Resistor_SMD:R_0402_1005Metric"
 			(at 121.412 69.85 90)
 			(effects
@@
 			)
 		)
-		(property "Footprint" ""
+		(property "Footprint" "Resistor_SMD:R_0402_1005Metric"
 			(at 160.782 92.71 90)
 			(effects
@@
 			)
 		)
-		(property "Footprint" ""
+		(property "Footprint" "Resistor_SMD:R_0402_1005Metric"
 			(at 173.482 128.27 90)
 			(effects
@@
 			)
 		)
-		(property "Footprint" ""
+		(property "Footprint" "Resistor_SMD:R_0402_1005Metric"
 			(at 173.482 115.57 90)
 			(effects
@@
 			)
 		)
-		(property "Footprint" ""
+		(property "Footprint" "Resistor_SMD:R_0402_1005Metric"
 			(at 160.782 110.49 90)
 			(effects
@@
 			)
 		)
-		(property "Footprint" ""
+		(property "Footprint" "Resistor_SMD:R_0402_1005Metric"
 			(at 151.892 92.71 90)
 			(effects
@@
 			)
 		)
-		(property "Footprint" ""
+		(property "Footprint" "Resistor_SMD:R_0402_1005Metric"
 			(at 121.412 87.63 90)
 			(effects
@@
 			)
 		)
-		(property "Footprint" ""
+		(property "Footprint" "Resistor_SMD:R_0402_1005Metric"
 			(at 130.302 69.85 90)
 			(effects
@@
 			)
 		)
-		(property "Footprint" ""
+		(property "Footprint" "Resistor_SMD:R_0402_1005Metric"
 			(at 143.002 92.71 90)
 			(effects
@@
 			)
 		)
-		(property "Footprint" ""
+		(property "Footprint" "Resistor_SMD:R_0402_1005Metric"
 			(at 143.002 110.49 90)
 			(effects
@@
 			)
 		)
-		(property "Footprint" ""
+		(property "Footprint" "Resistor_SMD:R_0402_1005Metric"
 			(at 112.522 87.63 90)
 			(effects
